File: ALUP_Receiver_Arduino.kicad_sch (KiCad schematic)
At the start: 9 parts, among them J1 Barrel_Jack_Switch, J2 5V LED, J3 D+ LED, J4 GND LED, U1 6N137

Commit message: Change pullup resistor
Parts:
- R2: value 2k -> 470
Changed lines of the file:
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@@
 			)
 		)
-		(property "Value" "2k"
+		(property "Value" "470"
 			(at 151.13 82.5499 0)
 			(effects
